File: kicad/base/buddy-base-v1.kicad_pcb (KiCad board)
At the start: 4 copper layers, 238.8 x 128.5 mm, 83 parts, among them J1 USB_C_Receptacle, J10 Conn_01x06_Socket, J11 Conn_01x06_Socket, J12 Conn_01x06_Socket, J13 Conn_01x06_Socket, J14 Conn_01x06_Socket, J15 Conn_01x06_Socket, J16 Conn_01x06_Socket, J17 Conn_01x06_Socket, J19 Conn_01x10_Socket, J2 Conn_01x02_Socket, J20 Conn_01x05, J3 Conn_01x06_Socket, J4 Conn_01x06_Socket, J5 Conn_01x06_Socket, J6 Conn_01x06_Socket, J7 Conn_01x06_Socket, J8 Conn_01x06_Socket, J9 Conn_01x06_Socket, Q2 AO3401A, SW1 SW_SPDT, U1 AP63203WU, U2 THVD1450DR

Commit message: Add Buddy Audio bus
Parts:
- removed D10, D11, D12, D13, D14, D15, D16, D5, D8, D9: LED, LED_SMD:LED_1206_3216Metric
- removed J19: Conn_01x10_Socket, Connector_PinSocket_2.54mm:PinSocket_1x10_P2.54mm_Vertical
- removed J20: Conn_01x05, Connector_PinHeader_2.54mm:PinHeader_1x05_P2.54mm_Vertical
- removed R10, R11, R12, R13, R14, R15, R16, R17, R18, R9: 470, Resistor_SMD:R_0603_1608Metric
- added C10: 10n, Capacitor_SMD:C_0402_1005Metric, F.Cu at (156.8, 56.9)
- added C11: 100n, Capacitor_SMD:C_0402_1005Metric, F.Cu at (156.8, 58.0)
- added C12: 1u, Capacitor_SMD:C_0402_1005Metric, F.Cu at (156.8, 59.1)
- added C13: 10n, Capacitor_SMD:C_0402_1005Metric, F.Cu at (141.7, 60.8)
- added C14: 100n, Capacitor_SMD:C_0402_1005Metric, F.Cu at (142.8, 60.8)
- added C15: 100n, Capacitor_SMD:C_0402_1005Metric, F.Cu at (155.3, 74.5)
- added C8: 1u, Capacitor_SMD:C_0402_1005Metric, F.Cu at (139.4, 66.9)
- added C9: 1u, Capacitor_SMD:C_0402_1005Metric, F.Cu at (140.6, 60.8)
- added J18: Conn_01x06, Connector_PinSocket_2.54mm:PinSocket_1x06_P2.54mm_Vertical, F.Cu at (248.7, 135.1)
- added R31: R, Resistor_SMD:R_0603_1608Metric, F.Cu at (141.7, 67.1)
- added R32: R, Resistor_SMD:R_0603_1608Metric, F.Cu at (144.4, 77.4)
- added R33: R, Resistor_SMD:R_0603_1608Metric, F.Cu at (155.6, 77.5)
- added U3: ICE40UP5K-SG48ITR, Package_DFN_QFN:QFN-48-1EP_7x7mm_P0.5mm_EP5.6x5.6mm, F.Cu at (150.0, 60.5)
- added U4: AP2127K-1.2, Package_TO_SOT_SMD:SOT-23-5, F.Cu at (141.7, 64.0)
- added U5: W25Q32JVSS, Package_SO:SOIC-8_5.3x5.3mm_P1.27mm, F.Cu at (150.0, 75.9)
- J15, J16, J17: value Conn_01x06_Socket -> Conn_01x06
- moved C7 187.7 mm to (233.9, 105.0), turned to -90 degrees
- moved R6 186.0 mm to (231.4, 105.8), turned to 180 degrees
- moved R7 182.0 mm to (230.3, 108.2), turned to 90 degrees
- moved R8 181.2 mm to (232.5, 108.2), turned to 90 degrees
- moved U2 181.2 mm to (231.7, 101.5), turned to -90 degrees
- moved J15 151.7 mm to (215.7, 96.8)
- moved R28 56.1 mm to (192.6, 31.5)
- moved R27 56.1 mm to (195.9, 31.5)
- moved R21 56.0 mm to (78.6, 31.5)
- moved R22 56.0 mm to (75.5, 31.5)
- moved R23 56.0 mm to (117.9, 31.5)
- moved R24 56.0 mm to (114.6, 31.5)
- moved R25 56.0 mm to (156.9, 31.5)
- moved R26 56.0 mm to (153.6, 31.5)
- moved R29 56.0 mm to (234.9, 31.5)
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Connections:
- J11 pad 1: SLOT_5 -> MCLK
- J11 pad 2: BUS_A -> BLCK
- J11 pad 3: BUS_B -> FSYNC
- J11 pad 4: 3V3_SYS -> S5_AUDIO_IN
- J11 pad 5: 5V_SYS -> S5_AUDIO_OUT
- J13 pad 1: SLOT_6 -> MCLK
- J13 pad 2: BUS_A -> BLCK
- J13 pad 3: BUS_B -> FSYNC
- J13 pad 4: 3V3_SYS -> S6_AUDIO_IN
- J13 pad 5: 5V_SYS -> S6_AUDIO_OUT
- J15 pad 1: PATCH -> RESET_1
- J15 pad 2: BUS_A -> BUS_TX
- J15 pad 3: BUS_B -> BUS_RX
- J16 pad 1: PATCH -> MCLK
- J16 pad 2: BUS_A -> BLCK
- J16 pad 3: BUS_B -> FSYNC
- J16 pad 4: 3V3_SYS -> TDM_TX
- J16 pad 5: 5V_SYS -> TDM_RX
- J17 pad 1: BUS_TX -> RESET_2
- J17 pad 2: BUS_RX -> BUS_TX
- J17 pad 3: BUS_EN -> BUS_RX
- J3 pad 1: SLOT_1 -> MCLK
- J3 pad 2: BUS_A -> BLCK
- J3 pad 3: BUS_B -> FSYNC
- J3 pad 4: 3V3_SYS -> S1_AUDIO_IN
- J3 pad 5: 5V_SYS -> S1_AUDIO_OUT
- J5 pad 1: SLOT_2 -> MCLK
- J5 pad 2: BUS_A -> BLCK
- J5 pad 3: BUS_B -> FSYNC
- J5 pad 4: 3V3_SYS -> S2_AUDIO_IN
- J5 pad 5: 5V_SYS -> S2_AUDIO_OUT
- J7 pad 1: SLOT_3 -> MCLK
- J7 pad 2: BUS_A -> BLCK
- J7 pad 3: BUS_B -> FSYNC
- J7 pad 4: 3V3_SYS -> S3_AUDIO_IN
- J7 pad 5: 5V_SYS -> S3_AUDIO_OUT
- J9 pad 1: SLOT_4 -> MCLK
- J9 pad 2: BUS_A -> BLCK
- J9 pad 3: BUS_B -> FSYNC
- J9 pad 4: 3V3_SYS -> S4_AUDIO_IN
- J9 pad 5: 5V_SYS -> S4_AUDIO_OUT
Routing:
- net BLCK: track 0.00 -> 386.3 mm, vias 0 -> 10
- net FSYNC: track 0.00 -> 382.8 mm, vias 0 -> 6
- net MCLK: track 0.00 -> 346.1 mm, vias 0 -> 5
- net BUS_A: track 525.6 -> 287.5 mm, vias 0 -> 1
- net BUS_B: track 528.6 -> 293.1 mm, vias 0 -> 1
- net PATCH: track 204.4 -> 0.00 mm
- net BUS_EN: track 204.1 -> 0.65 mm
- net BUS_RX: track 198.8 -> 35.3 mm
- net BUS_TX: track 199.8 -> 43.9 mm, vias 0 -> 2
- net S6_AUDIO_OUT: track 0.00 -> 114.5 mm
- net S6_AUDIO_IN: track 0.00 -> 110.9 mm
- net S1_AUDIO_IN: track 0.00 -> 106.6 mm
- net S1_AUDIO_OUT: track 0.00 -> 103.8 mm
- net RESET_1: track 0.00 -> 86.3 mm, vias 0 -> 4
- net S5_AUDIO_OUT: track 0.00 -> 73.6 mm
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Other:
- board text added: "BCLK"
- board text added: "BRAIN"
- board text added: "FSYNC"
- board text added: "MCLK"
- board text added: "RESET1"
- board text removed: "3V3"
- board text removed: "3V3_SYS"
- board text removed: "5V_SYS"
- board text removed: "EN"
- board text removed: "EXT PWR"
- board text removed: "OFF"
- board text removed: "ON"
- board text removed: "PATCH"
- board text removed: "V_OR"
