File: kicad/cards/knob-buddy/knob-buddy.kicad_pcb (KiCad board)
At the start: 2 copper layers, 38 x 64 mm, 25 parts, among them J1 Conn_01x06_Pin, J2 Conn_01x06_Pin, J3 Conn_01x05, J4 Conn_02x03_Odd_Even, U1 THVD1450DR, U2 STM32C011F4Px

Commit message: Update cards
Parts:
- J3: value Conn_01x05 -> Conn_ARM_SWD_TagConnect_TC2030-NL; footprint Connector_PinHeader_1.27mm:PinHeader_1x05_P1.27mm_Vertical -> Connector:Tag-Connect_TC2030-IDC-NL_2x03_P1.27mm_Vertical
- moved J3 2.22 mm to (125.2, 60.9), turned to 90 degrees
- moved RV2 0.71 mm to (149.5, 81.2)
- moved RV1 0.65 mm to (128.0, 81.1)
- moved J4 0.60 mm to (142.6, 105.2)
- moved RV4 0.35 mm to (149.5, 95.7)
- moved RV3 0.28 mm to (128.0, 95.6)
- moved RV5 0.13 mm to (128.0, 110.1)
- moved RV6 0.11 mm to (149.5, 110.2)
Connections:
- J1 pad 1: unconnected-(J1-Pin_1-Pad1) -> MCLK
- J1 pad 2: unconnected-(J1-Pin_2-Pad2) -> BLCK
- J1 pad 3: unconnected-(J1-Pin_3-Pad3) -> FSYNC
- J1 pad 4: +3V3 -> S4_AUDIO_IN
- J1 pad 5: unconnected-(J1-Pin_5-Pad5) -> S4_AUDIO_OUT
- J3 pad 3: SWCLK -> NRST
- J3 pad 4: NRST -> SWCLK
Routing:
- net +3V3: track 194.4 -> 164.3 mm
- net POT_2: track 54.5 -> 64.5 mm
- net POT_1: track 50.6 -> 56.1 mm, vias 2 -> 0
- net SWCLK: track 10.0 -> 15.3 mm
- net BUS_TX: track 8.67 -> 4.60 mm, vias 2 -> 0
- net SWDIO: track 9.34 -> 13.2 mm, vias 2 -> 0
- net NRST: track 19.9 -> 16.9 mm
- net POT_6: track 67.3 -> 64.4 mm
- net POT_4: track 60.6 -> 63.2 mm, vias 0 -> 1
- net POT_3: track 57.4 -> 59.4 mm, vias 2 -> 1
- net GND: track 19.5 -> 20.9 mm, vias 9 -> 10
- net POT_5: track 63.9 -> 62.9 mm, vias 0 -> 1
- net BUS_EN: track 4.77 -> 4.86 mm, vias 0 -> 2
Other:
- board text removed: "1"
- board text removed: "2"
- board text removed: "3"
- board text removed: "4"
- board text removed: "5"
- board text removed: "6"
- board text removed: "JLCJLCJLCJLC"
