File: kicad/cards/knob-buddy/knob-buddy.kicad_sch (KiCad schematic)
At the start: 18 parts, among them J1 Conn_01x06_Pin, J2 Conn_01x06_Pin, J3 Conn_01x05, U1 THVD1450DR, U2 STM32C011F4Px

Commit message: Update cards
Parts:
- removed J3: Conn_01x05, Connector_PinHeader_1.27mm:PinHeader_1x05_P1.27mm_Vertical, symbol Connector_Generic:Conn_01x05
- added J3: Conn_ARM_SWD_TagConnect_TC2030-NL, Connector:Tag-Connect_TC2030-IDC-NL_2x03_P1.27mm_Vertical, symbol Connector:Conn_ARM_SWD_TagConnect_TC2030-NL
Connections:
- net +3V3: now also J3.1 (VCC); no longer J1.4 (Pin_4)
- net GND: now also J3.5 (GND)
- net NRST: now also J3.3 (~{RESET})
- net SWCLK: now also J3.4 (SWCLK)
- net SWDIO: now also J3.2 (SWDIO)
- net MCLK: now reaches J1.1 (Pin_1)
- net BLCK: now reaches J1.2 (Pin_2)
- net FSYNC: now reaches J1.3 (Pin_3)
- net S4_AUDIO_OUT: now reaches J1.5 (Pin_5)
- new net S4_AUDIO_IN: J1.4 (Pin_4)
- no-connect marks 4 -> 1
