File: kicad/cards/line-buddy/buddy_sheet.kicad_sch (KiCad schematic)
At the start: 1 part

Commit message: Finish Line Buddy
Parts:
- added C10, C12, C13, C14, C7: 10u, Capacitor_SMD:C_0402_1005Metric, symbol Device:C
- added C11, C6, C9: 0.1u, Capacitor_SMD:C_0402_1005Metric, symbol Device:C
- added C15, C16, C17, C18: 47u, Capacitor_SMD:CP_Elec_6.3x5.4, symbol Device:C_Polarized
- added C8: 1u, Capacitor_SMD:C_0402_1005Metric, symbol Device:C
- added J4: AnalogIn, BuddySystem:PJ-358, symbol Connector_Audio:AudioJack3
- added J5: LineOut, BuddySystem:PJ-358, symbol Connector_Audio:AudioJack3
- added J6: HeadphoneOut, BuddySystem:PJ-358, symbol Connector_Audio:AudioJack3
- added R14, R15: 4.7K, Resistor_SMD:R_0603_1608Metric, symbol Device:R
- added R6, R7, R8, R9: 100K, Resistor_SMD:R_0603_1608Metric, symbol Device:R
- U3: value (none) -> TAC5112
Connections:
- net +3V3: now also U3.23 (AVDD), U3.6 (IOVDD), C10.2, C11.2, C12.2, C9.2, R14.2, R15.2
- net GND: now also U3.13 (ADDR), U3.25 (VSS), U3.A1 (VSS), U3.A2 (VSS), U3.A3 (VSS), U3.A4 (VSS), C10.1, C11.1, C12.1, C6.1, C7.1, C8.1, C9.1, J4.S, J5.S, J6.S, R6.2, R7.2, R8.2, R9.2
- net SCL: now also R14.1
- net SDA: now also R15.1
- net DREG: now reaches U3.1 (DREG)
- net DREG: now also C6.2, C7.2
- net IN1P: now reaches U3.15 (IN1P)
- net IN1P: now also C14.2, R7.1
- net IN1M: now reaches U3.16 (IN1M)
- net IN1M: now also R8.1
- net IN2P: now reaches U3.17 (IN2P)
- net IN2P: now also C13.2, R6.1
- net IN2M: now reaches U3.18 (IN2M)
- net IN2M: now also R9.1
- net OUT1M: now reaches U3.19 (OUT1M)
- net OUT1M: now also C17.1
- net OUT1P: now reaches U3.20 (OUT1P)
- net OUT1P: now also C15.1
- net OUT2P: now reaches U3.21 (OUT2P)
- net OUT2P: now also C16.1
- net OUT2M: now reaches U3.22 (OUT2M)
- net OUT2M: now also C18.1
- net VREF: now reaches U3.24 (VREF)
- net VREF: now also C8.2
- net AUDIO_IN renamed MOSI
- net AUDIO_OUT renamed MISO
- new net: C14.1, J4.T
- new net: C13.1, J4.R
- new net HP_OUT_L: C15.2, J6.T
- new net HP_OUT_R: C16.2, J6.R
- new net LINE_OUT_L: C17.2, J5.T
- new net LINE_OUT_R: C18.2, J5.R
- no-connect marks 0 -> 6
Other:
- moved on the sheet: U3
