File: kicad/cards/line-buddy/line-buddy.kicad_pcb (KiCad board)
At the start: 2 copper layers, 38 x 64 mm, 41 parts, among them J1 Conn_01x06_Pin, J2 Conn_01x06_Pin, J3 AudioJack3, J4 Conn_01x05, J5 AudioJack3, J6 AudioJack3, J7 Conn_01x04, U1 THVD1450DR, U2 STM32C011F4Px

Commit message: Add new line buddy WIP
Parts:
- removed C10: 4.7u, Capacitor_SMD:C_0402_1005Metric
- removed C11, C9: 100n, Capacitor_SMD:C_0402_1005Metric
- removed C12: 1u, Capacitor_SMD:C_0402_1005Metric
- removed C13, C14, C15, C18: 10u, Capacitor_SMD:C_0402_1005Metric
- removed C16, C17: 47u, Capacitor_SMD:C_0603_1608Metric
- removed C6, C7: 100n, Capacitor_SMD:C_0603_1608Metric
- removed J4: Conn_01x05, Connector_PinHeader_1.27mm:PinHeader_1x05_P1.27mm_Vertical
- removed J5, J6: AudioJack3, BuddySystem:PJ-358
- removed J7: Conn_01x04, Connector_PinHeader_2.54mm:PinHeader_1x04_P2.54mm_Vertical
- removed R12, R13: 4.7K, Resistor_SMD:R_0603_1608Metric
- removed R6, R7: 1K, Resistor_SMD:R_0603_1608Metric
- removed R8, R9: 100R, Resistor_SMD:R_0603_1608Metric
- J3: value AudioJack3 -> Conn_ARM_SWD_TagConnect_TC2030-NL; footprint BuddySystem:PJ-358 -> Connector:Tag-Connect_TC2030-IDC-NL_2x03_P1.27mm_Vertical
- U3: footprint BuddySystem:QFN-32_L5.0-W5.0-P0.50-TL-EP3.4 -> BuddySystem:VQFN-24_L4.0-W4.0-P0.50-BL-EP2.1_1
- moved J3 23.7 mm to (125.2, 60.9)
- moved U3 8.29 mm to (141.1, 108.0)
Connections:
- net CODEC_PH_DCT renamed SDA
- C2 pad 1: HPVDD -> +3V3
- C3 pad 1: HPVDD -> +3V3
- C5 pad 1: HPVDD -> +3V3
- J1 pad 1: unconnected-(J1-Pin_1-Pad1) -> MCLK
- J1 pad 2: unconnected-(J1-Pin_2-Pad2) -> BLCK
- J1 pad 3: unconnected-(J1-Pin_3-Pad3) -> FSYNC
- J1 pad 4: unconnected-(J1-Pin_4-Pad4) -> AUDIO_IN
- J1 pad 5: HPVDD -> AUDIO_OUT
- J2 pad 4: HPVDD -> +3V3
- R1 pad 2: HPVDD -> +3V3
- R4 pad 2: HPVDD -> +3V3
- U1 pad 8: HPVDD -> +3V3
- U2 pad 1: I2C_SDA -> unconnected-(U2-PB7-Pad1)
- U2 pad 15: CODEC_RST -> unconnected-(U2-PA8-Pad15)
- U2 pad 20: I2C_SCL -> unconnected-(U2-PB6-Pad20)
- U2 pad 4: HPVDD -> +3V3
- U3 pad 10: I2C_SDA -> unconnected-(U3-GPIO2-Pad10)
- U3 pad 12: GND -> unconnected-(U3-GPI1-Pad12)
- U3 pad 13: LINE_IN_L -> unconnected-(U3-ADDR-Pad13)
- U3 pad 14: LINE_IN_R -> unconnected-(U3-MICBIAS-Pad14)
- U3 pad 17: GND -> unconnected-(U3-IN2P-Pad17)
- U3 pad 18: Net-(U3-REF) -> unconnected-(U3-IN2M-Pad18)
- U3 pad 2: CODEC_BCLK -> BLCK
- U3 pad 22: LINE_OUT_L -> unconnected-(U3-OUT2M-Pad22)
- U3 pad 23: LINE_OUT_R -> unconnected-(U3-AVDD-Pad23)
- U3 pad 24: Net-(U3-AVDD) -> unconnected-(U3-VREF-Pad24)
- U3 pad 25: PHONE_OUT_L -> unconnected-(U3-VSS-Pad25)
- U3 pad 3: CODEC_WCLK -> FSYNC
- U3 pad 4: CODEC_DIN -> AUDIO_OUT
- U3 pad 5: CODEC_DOUT -> AUDIO_IN
- U3 pad 6: HPVDD -> unconnected-(U3-IOVDD-Pad6)
- U3 pad 7: GND -> SCL
- U3 pad 9: I2C_SCL -> unconnected-(U3-GPIO1-Pad9)
Routing:
- net HPVDD: track 180.0 -> 0.00 mm
- net +3V3: track 0.00 -> 60.2 mm
- net I2C_SCL: track 47.5 -> 0.00 mm, vias 2 -> 0
- net CODEC_RST: track 42.0 -> 0.00 mm, vias 2 -> 0
- net I2C_SDA: track 39.5 -> 0.00 mm, vias 2 -> 0
- net PHONE_OUT_R: track 37.1 -> 0.00 mm, vias 2 -> 0
- net LINE_IN_R: track 36.2 -> 0.00 mm
- net LINE_OUT_R: track 25.1 -> 0.00 mm, vias 2 -> 0
- net PHONE_OUT_L: track 20.4 -> 0.00 mm, vias 2 -> 0
- net LINE_IN_L: track 19.4 -> 0.00 mm
- net GND: track 31.0 -> 20.9 mm, vias 20 -> 10
- net CODEC_DOUT: track 8.93 -> 0.00 mm
- net CODEC_BCLK: track 8.74 -> 0.00 mm
- net LINE_OUT_L: track 8.19 -> 0.00 mm, vias 2 -> 0
- net CODEC_DIN: track 8.09 -> 0.00 mm
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Other:
- board text removed: "LINE IN"
- board text removed: "LINE OUT"
- board text removed: "PHONES"

Commit message: Finish Line Buddy
Parts:
- added C10: 10u, Capacitor_SMD:C_0402_1005Metric, F.Cu at (145.3, 110.9)
- added C11: 0.1u, Capacitor_SMD:C_0402_1005Metric, F.Cu at (136.2, 106.5)
- added C12: 10u, Capacitor_SMD:C_0402_1005Metric, F.Cu at (136.2, 107.7)
- added C13: 10u, Capacitor_SMD:C_0402_1005Metric, F.Cu at (130.1, 71.6)
- added C14: 10u, Capacitor_SMD:C_0402_1005Metric, F.Cu at (130.1, 69.6)
- added C15: 47u, Capacitor_SMD:CP_Elec_6.3x5.4, F.Cu at (129.2, 94.9)
- added C16: 47u, Capacitor_SMD:CP_Elec_6.3x5.4, F.Cu at (137.3, 94.9)
- added C17: 47u, Capacitor_SMD:CP_Elec_6.3x5.4, F.Cu at (145.4, 94.9)
- added C18: 47u, Capacitor_SMD:CP_Elec_6.3x5.4, F.Cu at (153.6, 94.9)
- added C6: 0.1u, Capacitor_SMD:C_0402_1005Metric, F.Cu at (137.0, 109.9)
- added C7: 10u, Capacitor_SMD:C_0402_1005Metric, F.Cu at (137.0, 111.0)
- added C8: 1u, Capacitor_SMD:C_0402_1005Metric, F.Cu at (136.2, 108.8)
- added C9: 0.1u, Capacitor_SMD:C_0402_1005Metric, F.Cu at (145.3, 109.9)
- added J4: AnalogIn, BuddySystem:PJ-358, F.Cu at (128.3, 83.2)
- added J5: LineOut, BuddySystem:PJ-358, F.Cu at (140.7, 83.2)
- added J6: HeadphoneOut, BuddySystem:PJ-358, F.Cu at (153.3, 83.2)
- added R14: 4.7K, Resistor_SMD:R_0603_1608Metric, F.Cu at (146.3, 108.3)
- added R15: 4.7K, Resistor_SMD:R_0603_1608Metric, F.Cu at (146.3, 106.8)
- added R6: 100K, Resistor_SMD:R_0603_1608Metric, F.Cu at (127.3, 71.6)
- added R7: 100K, Resistor_SMD:R_0603_1608Metric, F.Cu at (127.3, 69.6)
- added R8: 100K, Resistor_SMD:R_0603_1608Metric, F.Cu at (141.1, 103.5)
- added R9: 100K, Resistor_SMD:R_0603_1608Metric, F.Cu at (139.5, 103.5)
- U3: value ~ -> TAC5112
- moved U3 0.08 mm to (141.2, 108.0)
Connections:
- net AUDIO_IN renamed MOSI
- net AUDIO_OUT renamed MISO
- C2 pad 1: +3V3 -> AVDD
- C3 pad 1: +3V3 -> AVDD
- C5 pad 1: +3V3 -> AVDD
- J2 pad 4: +3V3 -> AVDD
- J3 pad 1: +3V3 -> AVDD
- R1 pad 2: +3V3 -> AVDD
- R4 pad 2: +3V3 -> AVDD
- U1 pad 8: +3V3 -> AVDD
- U2 pad 1: unconnected-(U2-PB7-Pad1) -> SDA
- U2 pad 20: unconnected-(U2-PB6-Pad20) -> SCL
- U2 pad 4: +3V3 -> AVDD
- U3 pad 1: unconnected-(U3-DREG-Pad1) -> DREG
- U3 pad 13: unconnected-(U3-ADDR-Pad13) -> GND
- U3 pad 15: unconnected-(U3-IN1P-Pad15) -> IN1P
- U3 pad 16: unconnected-(U3-IN1M-Pad16) -> IN1M
- U3 pad 17: unconnected-(U3-IN2P-Pad17) -> IN2P
- U3 pad 18: unconnected-(U3-IN2M-Pad18) -> IN2M
- U3 pad 19: unconnected-(U3-OUT1M-Pad19) -> OUT1M
- U3 pad 20: unconnected-(U3-OUT1P-Pad20) -> OUT1P
- U3 pad 21: unconnected-(U3-OUT2P-Pad21) -> OUT2P
- U3 pad 22: unconnected-(U3-OUT2M-Pad22) -> OUT2M
- U3 pad 23: unconnected-(U3-AVDD-Pad23) -> AVDD
- U3 pad 24: unconnected-(U3-VREF-Pad24) -> VREF
- U3 pad 25: unconnected-(U3-VSS-Pad25) -> GND
- U3 pad 6: unconnected-(U3-IOVDD-Pad6) -> AVDD
- U3 pad A1: unconnected-(U3-VSS-PadA1) -> GND
- U3 pad A2: unconnected-(U3-VSS-PadA2) -> GND
- U3 pad A3: unconnected-(U3-VSS-PadA3) -> GND
- U3 pad A4: unconnected-(U3-VSS-PadA4) -> GND
Routing:
- net AVDD: track 0.00 -> 148.4 mm, vias 0 -> 2
- net SCL: track 0.00 -> 74.4 mm, vias 0 -> 2
- net SDA: track 0.00 -> 67.1 mm
- net IN1P: track 0.00 -> 64.5 mm
- net +3V3: track 60.2 -> 0.00 mm
- net IN2P: track 0.00 -> 50.4 mm
- net HP_OUT_L: track 0.00 -> 29.8 mm, vias 0 -> 1
- net HP_OUT_R: track 0.00 -> 23.3 mm, vias 0 -> 1
- net OUT2M: track 0.00 -> 22.0 mm, vias 0 -> 2
- net GND: track 20.9 -> 41.6 mm, vias 10 -> 26
- net Net-(C14-Pad1): track 0.00 -> 19.0 mm
- net LINE_OUT_R: track 0.00 -> 17.5 mm
- net OUT1M: track 0.00 -> 15.0 mm, vias 0 -> 2
- net OUT1P: track 0.00 -> 14.4 mm, vias 0 -> 2
- net OUT2P: track 0.00 -> 11.3 mm, vias 0 -> 2
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Other:
- board text added: "HEAD"
- board text added: "IN"
- board text added: "LINE"
- board text added: "OUT"
- board text added: "PHONE"
